Commit message: Working urdf.xacro in rviz2 with tf2 transforms.

File: src/glados_description/urdf/glados.urdf.xacro (robot description, xacro)
@@ -7,5 +7,5 @@
   <xacro:property name="body_width" value="0.050" />
   <xacro:property name="body_length" value="0.035" />
-  <gazebo reference="glados_body">
+  <gazebo reference="base_link">
     <material>Gazebo/White</material>
     <mu1>0.2</mu1>
@@ -22,5 +22,5 @@
     <mu2>0.84</mu2>
   </gazebo>
-  <link name="glados_body">
+  <link name="base_link">
     <visual>
       <geometry>
@@ -71,5 +71,5 @@
   </link>
   <joint name="jointL" type="continuous">
-    <parent link="glados_body"/>
+    <parent link="base_link"/>
     <child link="wheelL"/>
     <axis xyz="0 0 1"/>
@@ -78,5 +78,5 @@
   </joint>
   <joint name="jointR" type="continuous">
-    <parent link="glados_body"/>
+    <parent link="base_link"/>
     <child link="wheelR"/>
     <axis xyz="0 0 1"/>

Commit message: wip adding castor

File: src/glados_description/urdf/glados.urdf.xacro (robot description, xacro)
@@ -4,4 +4,5 @@
   <xacro:property name="wheel_radius" value="0.034" />
   <xacro:property name="wheel_width" value="0.010" />
+  <xacro:property name="castor_radius" value="0.005" />
   <xacro:property name="body_height" value="0.1" />
   <xacro:property name="body_width" value="0.050" />
@@ -70,4 +71,20 @@
     </inertial>
   </link>
+  <link name="castor">
+    <visual>
+      <geometry>
+        <sphere radius="${castor_radius}"/>
+      </geometry>
+    </visual>
+    <collision>
+      <geometry>
+        <sphere radius="${castor_radius}"/>
+      </geometry>
+    </collision>
+    <inertial>
+      <mass value="0.05"/>
+      <inertia ixx="1.75e-5" ixy="0.0" ixz="0.0" iyy="1.75e-5" iyz="0.0" izz="1.75e-5"/>
+    </inertial>
+  </link>
   <joint name="jointL" type="continuous">
     <parent link="base_link"/>
@@ -84,4 +101,11 @@
     <dynamics friction="0.1"/>
   </joint>
+  <joint name="jointCastor" type="continuous">
+    <parent link="base_link"/>
+    <child link="castor"/>
+    <axis xyz="0 0 1"/>
+    <origin xyz="${body_length/2} 0 ${body_height*7/8 - body_height/2}" rpy="${pi/2} 0 0" />
+    <dynamics friction="0.1"/>
+  </joint>
   <!-- <gazebo>
     <plugin name="wb_plugin" filename="libwb_plugin.so"> </plugin>

Commit message: wip.

File: src/glados_description/urdf/glados.urdf.xacro (robot description, xacro)
@@ -71,5 +71,5 @@
     </inertial>
   </link>
-  <link name="castor">
+  <!-- <link name="castor">
     <visual>
       <geometry>
@@ -86,5 +86,5 @@
       <inertia ixx="1.75e-5" ixy="0.0" ixz="0.0" iyy="1.75e-5" iyz="0.0" izz="1.75e-5"/>
     </inertial>
-  </link>
+  </link> -->
   <joint name="jointL" type="continuous">
     <parent link="base_link"/>
@@ -101,5 +101,5 @@
     <dynamics friction="0.1"/>
   </joint>
-  <joint name="jointCastor" type="continuous">
+  <!-- <joint name="jointCastor" type="continuous">
     <parent link="base_link"/>
     <child link="castor"/>
@@ -107,5 +107,5 @@
     <origin xyz="${body_length/2} 0 ${body_height*7/8 - body_height/2}" rpy="${pi/2} 0 0" />
     <dynamics friction="0.1"/>
-  </joint>
+  </joint> -->
   <!-- <gazebo>
     <plugin name="wb_plugin" filename="libwb_plugin.so"> </plugin>

Commit message: Trying to get the controller working. wip

File: src/glados_description/urdf/glados.urdf.xacro (robot description, xacro)
@@ -23,4 +23,10 @@
     <mu2>0.84</mu2>
   </gazebo> -->
+  <!-- <link name="base_footprint"/>
+  <joint name="base_joint" type="fixed">
+    <parent link="base_footprint"/>
+    <child link="base_link"/>
+    <origin xyz="0.0 0.0 0.10" rpy="0 0 0"/>
+  </joint> -->
   <link name="base_link">
     <visual>

Commit message: Try out robleo in my own simulation.

File: src/glados_description/urdf/glados.urdf.xacro (robot description, xacro)
@@ -8,20 +8,4 @@
   <xacro:property name="body_width" value="0.050" />
   <xacro:property name="body_length" value="0.035" />
-  <!-- <gazebo reference="base_link">
-    <material>Gazebo/White</material>
-    <mu1>0.2</mu1>
-    <mu2>0.2</mu2>
-  </gazebo>
-  <gazebo reference="wheelR">
-    <material>Gazebo/Red</material>
-    <mu1>0.84</mu1>
-    <mu2>0.84</mu2>
-  </gazebo>
-  <gazebo reference="wheelL">
-    <material>Gazebo/Blue</material>
-    <mu1>0.84</mu1>
-    <mu2>0.84</mu2>
-  </gazebo> -->
-  <!-- <link name="base_footprint"/>
   <joint name="base_joint" type="fixed">
     <parent link="base_footprint"/>
@@ -114,6 +98,3 @@
     <dynamics friction="0.1"/>
   </joint> -->
-  <!-- <gazebo>
-    <plugin name="wb_plugin" filename="libwb_plugin.so"> </plugin>
-  </gazebo> -->
 </robot>

Commit message: Fix URDF.

File: src/glados_description/urdf/glados.urdf.xacro (robot description, xacro)
@@ -8,4 +8,5 @@
   <xacro:property name="body_width" value="0.050" />
   <xacro:property name="body_length" value="0.035" />
+  <!-- <link name="base_footprint"/>
   <joint name="base_joint" type="fixed">
     <parent link="base_footprint"/>

Commit message: Turn collision off such that friction is no loger a problem

File: src/glados_description/urdf/glados.urdf.xacro (robot description, xacro)
@@ -20,9 +20,9 @@
       </geometry>
     </visual>
-    <collision>
+    <!-- <collision>
       <geometry>
         <box size="${body_length} ${body_width} ${body_height}"/>
       </geometry>
-    </collision>
+    </collision> -->
     <inertial>
       <mass value="0.18"/>

Commit message: Change body size to more easily check the axis and directions of travel. Also start rotated to point to the right direction and update wheel rotation axis in URDF, because they were wrong.

File: src/glados_description/urdf/glados.urdf.xacro (robot description, xacro)
@@ -5,7 +5,7 @@
   <xacro:property name="wheel_width" value="0.010" />
   <xacro:property name="castor_radius" value="0.005" />
-  <xacro:property name="body_height" value="0.1" />
-  <xacro:property name="body_width" value="0.050" />
-  <xacro:property name="body_length" value="0.035" />
+  <xacro:property name="body_height" value="0.05" />
+  <xacro:property name="body_width" value="0.05" />
+  <xacro:property name="body_length" value="0.1" />
   <!-- <link name="base_footprint"/>
   <joint name="base_joint" type="fixed">
@@ -20,9 +20,9 @@
       </geometry>
     </visual>
-    <!-- <collision>
+    <collision>
       <geometry>
         <box size="${body_length} ${body_width} ${body_height}"/>
       </geometry>
-    </collision> -->
+    </collision>
     <inertial>
       <mass value="0.18"/>
@@ -82,5 +82,5 @@
     <child link="wheelL"/>
     <axis xyz="0 0 1"/>
-    <origin xyz="0 ${body_width/2 + wheel_width/2} -${body_height/2 - 0.01}" rpy="${pi/2} 0 0" />
+    <origin xyz="0 ${body_width/2 + wheel_width/2} 0" rpy="-${pi/2} 0 0" />
     <dynamics friction="0.1"/>
   </joint>
@@ -89,5 +89,5 @@
     <child link="wheelR"/>
     <axis xyz="0 0 1"/>
-    <origin xyz="0 -${body_width/2 + wheel_width/2} -${body_height/2 - 0.01}" rpy="${pi/2} 0 0" />
+    <origin xyz="0 -${body_width/2 + wheel_width/2} 0" rpy="-${pi/2} 0 0" />
     <dynamics friction="0.1"/>
   </joint>

Commit message: Add test code to find bug. Allows more easy switching between glados and robleo.

File: src/glados_description/urdf/glados.urdf.xacro (robot description, xacro)
@@ -8,7 +8,7 @@
   <xacro:property name="body_width" value="0.05" />
   <xacro:property name="body_length" value="0.1" />
-  <!-- <link name="base_footprint"/>
+  <!-- <link name="odom"/>
   <joint name="base_joint" type="fixed">
-    <parent link="base_footprint"/>
+    <parent link="odom"/>
     <child link="base_link"/>
     <origin xyz="0.0 0.0 0.10" rpy="0 0 0"/>
@@ -16,10 +16,16 @@
   <link name="base_link">
     <visual>
+      <origin xyz="0 0 0" rpy="0 0 0" />
       <geometry>
+        <!-- <cylinder radius="0.025" length="0.03"/> -->
         <box size="${body_length} ${body_width} ${body_height}"/>
       </geometry>
+      <material name="Cyan">
+        <color rgba="0 1.0 1.0 1.0"/>
+      </material>
     </visual>
     <collision>
       <geometry>
+        <!-- <cylinder radius="0.025" length="0.03"/> -->
         <box size="${body_length} ${body_width} ${body_height}"/>
       </geometry>

File: src/glados_description/urdf/robleo.urdf.xacro (robot description, xacro)
@@ -1,11 +1,11 @@
 <?xml version="1.0" ?>
-<robot name="glados"
+<robot name="robleo"
   xmlns:xacro="http://ros.org/wiki/xacro">
-  <link name="base_footprint"/>
+  <!-- <link name="base_footprint"/>
   <joint name="base_joint" type="fixed">
     <parent link="base_footprint"/>
     <child link="base_link"/>
     <origin xyz="0.0 0.0 0.10" rpy="0 0 0"/>
-  </joint>
+  </joint> -->
   <link name="base_link">
     <visual>
@@ -30,11 +30,11 @@
     </inertial>
   </link>
-  <joint name="jointL" type="continuous">
+  <joint name="wheel_left_joint" type="continuous">
     <parent link="base_link"/>
-    <child link="wheelL"/>
+    <child link="wheel_left_link"/>
     <origin xyz="0.0 0.25 0.0" rpy="-1.57 0 0"/>
     <axis xyz="0 0 1"/>
   </joint>
-  <link name="wheelL">
+  <link name="wheel_left_link">
     <visual>
       <origin xyz="0 0 0" rpy="0 0 0" />
@@ -58,11 +58,11 @@
     </inertial>
   </link>
-  <joint name="jointR" type="continuous">
+  <joint name="wheel_right_joint" type="continuous">
     <parent link="base_link"/>
-    <child link="wheelR"/>
-    <origin xyz="0.0 -0.25 0.0" rpy="1.57 0 0"/>
+    <child link="wheel_right_link"/>
+    <origin xyz="0.0 -0.25 0.0" rpy="-1.57 0 0"/>
     <axis xyz="0 0 1"/>
   </joint>
-  <link name="wheelR">
+  <link name="wheel_right_link">
     <visual>
       <origin xyz="0 0 0" rpy="0 0 0"/>

Commit message: Test URDF's.

File: src/glados_description/urdf/glados.urdf.xacro (robot description, xacro)
@@ -18,6 +18,6 @@
       <origin xyz="0 0 0" rpy="0 0 0" />
       <geometry>
-        <!-- <cylinder radius="0.025" length="0.03"/> -->
-        <box size="${body_length} ${body_width} ${body_height}"/>
+        <cylinder radius="0.025" length="0.03"/>
+        <!-- <box size="${body_length} ${body_width} ${body_height}"/> -->
       </geometry>
       <material name="Cyan">
@@ -27,6 +27,6 @@
     <collision>
       <geometry>
-        <!-- <cylinder radius="0.025" length="0.03"/> -->
-        <box size="${body_length} ${body_width} ${body_height}"/>
+        <cylinder radius="0.025" length="0.03"/>
+        <!-- <box size="${body_length} ${body_width} ${body_height}"/> -->
       </geometry>
     </collision>

Commit message: Migrate to galactic and fix body visualization.

File: src/glados_description/urdf/glados.urdf.xacro (robot description, xacro)
@@ -18,6 +18,6 @@
       <origin xyz="0 0 0" rpy="0 0 0" />
       <geometry>
-        <cylinder radius="0.025" length="0.03"/>
-        <!-- <box size="${body_length} ${body_width} ${body_height}"/> -->
+        <!-- <cylinder radius="0.025" length="0.03"/> -->
+        <box size="${body_length} ${body_width} ${body_height}"/>
       </geometry>
       <material name="Cyan">
@@ -27,6 +27,6 @@
     <collision>
       <geometry>
-        <cylinder radius="0.025" length="0.03"/>
-        <!-- <box size="${body_length} ${body_width} ${body_height}"/> -->
+        <!-- <cylinder radius="0.025" length="0.03"/> -->
+        <box size="${body_length} ${body_width} ${body_height}"/>
       </geometry>
     </collision>

Commit message: Fixing a sudo apt upgrade.

File: src/glados_description/urdf/glados.urdf.xacro (robot description, xacro)
@@ -38,4 +38,5 @@
   <link name="wheelL">
     <visual>
+    <!-- <origin xyz="0 0 0" rpy="${pi/2} 0 0"/> -->
       <geometry>
         <cylinder length="${wheel_width}" radius="${wheel_radius}"/>
@@ -54,4 +55,5 @@
   <link name="wheelR">
     <visual>
+    <!-- <origin xyz="0 0 0" rpy="${pi/2} 0 0"/> -->
       <geometry>
         <cylinder length="${wheel_width}" radius="${wheel_radius}"/>
@@ -88,5 +90,5 @@
     <child link="wheelL"/>
     <axis xyz="0 0 1"/>
-    <origin xyz="0 ${body_width/2 + wheel_width/2} 0" rpy="-${pi/2} 0 0" />
+    <origin xyz="0 ${body_width/2 + wheel_width/2} 0" rpy="-1.57 0 0" />
     <dynamics friction="0.1"/>
   </joint>
@@ -95,5 +97,5 @@
     <child link="wheelR"/>
     <axis xyz="0 0 1"/>
-    <origin xyz="0 -${body_width/2 + wheel_width/2} 0" rpy="-${pi/2} 0 0" />
+    <origin xyz="0 -${body_width/2 + wheel_width/2} 0" rpy="-1.57 0 0" />
     <dynamics friction="0.1"/>
   </joint>
